Commit message: fixed urdf path-links

File: resources/shadow_hand_ign/urdf/shadow_hand.urdf (robot description, URDF)
Before this commit: robot shadow_hand, 25 links, 24 joints
Links:
- link forearm: geometry collision mesh filename=../shadow_hand/meshes/collision/forearm.stl; visual mesh filename=../shadow_hand/meshes/visual/forearm.dae
- link index_finger_distal: geometry collision mesh filename=../shadow_hand/meshes/collision/finger_distal.stl; visual mesh filename=../shadow_hand/meshes/visual/finger_distal.dae
- link index_finger_knuckle: geometry collision mesh filename=../shadow_hand/meshes/collision/knuckle.stl; visual mesh filename=../shadow_hand/meshes/visual/knuckle.dae
- link index_finger_middle: geometry collision mesh filename=../shadow_hand/meshes/collision/finger_middle.stl; visual mesh filename=../shadow_hand/meshes/visual/finger_middle.dae
- link index_finger_proximal: geometry collision mesh filename=../shadow_hand/meshes/collision/finger_proximal.stl; visual mesh filename=../shadow_hand/meshes/visual/finger_proximal.dae
- link little_finger_distal: geometry collision mesh filename=../shadow_hand/meshes/collision/finger_distal.stl; visual mesh filename=../shadow_hand/meshes/visual/finger_distal.dae
- link little_finger_knuckle: geometry collision mesh filename=../shadow_hand/meshes/collision/knuckle.stl; visual mesh filename=../shadow_hand/meshes/visual/knuckle.dae
- link little_finger_metacarpal: geometry collision mesh filename=../shadow_hand/meshes/collision/metacarpal.stl; visual mesh filename=../shadow_hand/meshes/visual/metacarpal.dae
- link little_finger_middle: geometry collision mesh filename=../shadow_hand/meshes/collision/finger_middle.stl; visual mesh filename=../shadow_hand/meshes/visual/finger_middle.dae
- link little_finger_proximal: geometry collision mesh filename=../shadow_hand/meshes/collision/finger_proximal.stl; visual mesh filename=../shadow_hand/meshes/visual/finger_proximal.dae
- link middle_finger_distal: geometry collision mesh filename=../shadow_hand/meshes/collision/finger_distal.stl; visual mesh filename=../shadow_hand/meshes/visual/finger_distal.dae
- link middle_finger_knuckle: geometry collision mesh filename=../shadow_hand/meshes/collision/knuckle.stl; visual mesh filename=../shadow_hand/meshes/visual/knuckle.dae
- link middle_finger_middle: geometry collision mesh filename=../shadow_hand/meshes/collision/finger_middle.stl; visual mesh filename=../shadow_hand/meshes/visual/finger_middle.dae
- link middle_finger_proximal: geometry collision mesh filename=../shadow_hand/meshes/collision/finger_proximal.stl; visual mesh filename=../shadow_hand/meshes/visual/finger_proximal.dae
- link palm: geometry collision mesh filename=../shadow_hand/meshes/collision/palm.stl; visual mesh filename=../shadow_hand/meshes/visual/palm.dae
- link ring_finger_distal: geometry collision mesh filename=../shadow_hand/meshes/collision/finger_distal.stl; visual mesh filename=../shadow_hand/meshes/visual/finger_distal.dae
- link ring_finger_knuckle: geometry collision mesh filename=../shadow_hand/meshes/collision/knuckle.stl; visual mesh filename=../shadow_hand/meshes/visual/knuckle.dae
- link ring_finger_middle: geometry collision mesh filename=../shadow_hand/meshes/collision/finger_middle.stl; visual mesh filename=../shadow_hand/meshes/visual/finger_middle.dae
- link ring_finger_proximal: geometry collision mesh filename=../shadow_hand/meshes/collision/finger_proximal.stl; visual mesh filename=../shadow_hand/meshes/visual/finger_proximal.dae
- link thumb_distal: geometry collision mesh filename=../shadow_hand/meshes/collision/thumb_distal.stl; visual mesh filename=../shadow_hand/meshes/visual/thumb_distal.dae
- link thumb_middle: geometry collision mesh filename=../shadow_hand/meshes/collision/thumb_middle.stl; visual mesh filename=../shadow_hand/meshes/visual/thumb_middle.dae
- link thumb_proximal: geometry collision mesh filename=../shadow_hand/meshes/collision/thumb_proximal.stl; visual mesh filename=../shadow_hand/meshes/visual/thumb_proximal.dae
- link wrist: geometry collision mesh filename=../shadow_hand/meshes/collision/wrist.stl; visual mesh filename=../shadow_hand/meshes/visual/wrist.dae
